File: SolarLader.kicad_sch (KiCad schematic)
At the start: 24 parts, among them J1 Conn_01x02, J2 UKDBBTAAA, J3 Conn_01x02, Q1 Q_PMOS_GSD, U1 BQ25185DLHR

Commit message: ReleaseCandidate1
Parts:
- removed H1, H2: MountingHole, MountingHole:MountingHole_2.2mm_M2, symbol Mechanical:MountingHole
- added H3, H4: MountingHole_Pad, MountingHole:MountingHole_2.2mm_M2_DIN965_Pad, symbol Mechanical:MountingHole_Pad
- added J4: Conn_01x06, Connector_PinHeader_1.00mm:PinHeader_1x06_P1.00mm_Vertical, symbol Connector_Generic:Conn_01x06
- added R9: 0, symbol Device:R
- R4: value 13k -> 5k
- R5: value 600 -> 1k
Connections:
- net +BATT: now also J4.3 (Pin_3)
- net GND: now also H3.1, H4.1, J4.6 (Pin_6)
- net Solar: now also J4.5 (Pin_5)
- net VIN: now also J4.2 (Pin_2), R9.1; no longer Q1.1 (G), R8.1
- net VSYS: now also J4.1 (Pin_1)
- new net Gate: J4.4 (Pin_4), Q1.1 (G), R8.1, R9.2
Other:
- note added: "1 kOhm => 300mA charching current"
- note added: "6kOhm ILIM = 500 mA VSET = 4.2V (Max Batt)"
- note removed: "13kOhm ILIM = 1100 mA VSET = 4.2V (Max Batt)"
- note removed: "600 Ohm => 500mA charching current"
- moved on the sheet: J3, Q1, R8
