File: SolarLaderWithAnaloge.kicad_pcb (KiCad board)
At the start: 2 copper layers, 26 x 18 mm, 33 parts, among them J1 Conn_01x04, J2 Conn_01x02, J3 Conn_01x01, J4 UKDBBTAAA, J5 Conn_01x02, Q1 AO3401A, U1 BQ25185DLHR, U2 LM66200DRLR

Commit message: Update the Jumper for the input
Parts:
- removed JP4: SolderJumper_2_Open, Jumper:SolderJumper-2_P1.3mm_Open_Pad1.0x1.5mm
- added JP5: SolderJumper_3_Bridged12, Jumper:SolderJumper-3_P1.3mm_Bridged12_Pad1.0x1.5mm, B.Cu at (135.8, 68.4)
- JP3: value SolderJumper_2_Open -> SolderJumper_3_Bridged12; footprint Jumper:SolderJumper-2_P1.3mm_Open_Pad1.0x1.5mm -> Jumper:SolderJumper-3_P1.3mm_Bridged12_Pad1.0x1.5mm
- moved JP3 0.56 mm to (135.8, 71.4), turned to 0 degrees
Connections:
- D3 pad 2: /J_Solar -> /DiodeSolar
- D4 pad 2: /J_VBUS -> /DiodeVBUS
- JP3 pad 1: /J_VBUS -> /LMVBUS
- U2 pad 3: /Solar -> /LMSolar
- U2 pad 6: VBUS -> /LMVBUS
Routing:
- net /DiodeVBUS: track 0.00 -> 4.48 mm, vias 0 -> 1
- net /J_VBUS: track 4.06 -> 0.00 mm, vias 1 -> 0
- net /DiodeSolar: track 0.00 -> 3.80 mm, vias 0 -> 1
- net /LMSolar: track 0.00 -> 3.36 mm, vias 0 -> 1
- net /LMVBUS: track 0.00 -> 3.24 mm, vias 0 -> 1
- net /Solar: track 8.17 -> 5.15 mm, vias 1 -> 0
- net /J_Solar: track 2.13 -> 0.00 mm, vias 1 -> 0
- net VBUS: track 9.26 -> 8.10 mm
- net GND: vias 17 -> 16
Other:
- board text added: "D"
- board text added: "U"
